File: MRDT_Rover_Controller/Controller Board/Controller Board.kicad_pcb (KiCad board)
At the start: 2 copper layers, 137.6 x 81.5 mm, 30 parts, among them Q1 S8050, SW1 EG1218, U1 MCP3008

Commit message: PCB Updated
Routing:
- net RightVert: track 17.6 -> 77.8 mm, vias 1 -> 2
- net RightHorz: track 14.9 -> 71.0 mm, vias 1 -> 2
- net RGHT_SEL: track 44.2 -> 93.3 mm, vias 1 -> 2
Changed lines of the file:
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@@
     (thickness 1.6)
     (drawings 25)
-    (tracks 460)
+    (tracks 499)
     (zones 0)
     (modules 30)
@@
   (segment (start 186.0296 106.337165) (end 186.0296 120.2944) (width 0.381) (layer B.Cu) (net 48))
   (segment (start 186.0296 120.2944) (end 186.0296 120.2944) (width 0.381) (layer B.Cu) (net 48))
-  (via (at 186.0296 120.2944) (size 0.8) (drill 0.4) (layers F.Cu B.Cu) (net 48))
+  (segment (start 186.0296 120.2944) (end 186.0296 123.7488) (width 0.381) (layer B.Cu) (net 48))
+  (segment (start 186.0296 123.7488) (end 186.0296 124.1552) (width 0.381) (layer B.Cu) (net 48))
+  (segment (start 186.0296 124.1552) (end 186.0296 124.1552) (width 0.381) (layer B.Cu) (net 48))
+  (via (at 186.0296 124.1552) (size 0.8) (drill 0.4) (layers F.Cu B.Cu) (net 48))
+  (segment (start 185.629601 123.755201) (end 163.226801 123.755201) (width 0.381) (layer F.Cu) (net 48))
+  (segment (start 186.0296 124.1552) (end 185.629601 123.755201) (width 0.381) (layer F.Cu) (net 48))
+  (segment (start 157.354274 123.945618) (end 155.2956 121.886944) (width 0.381) (layer F.Cu) (net 48))
+  (segment (start 162.634923 123.945619) (end 157.354274 123.945618) (width 0.381) (layer F.Cu) (net 48))
+  (segment (start 163.226801 123.755201) (end 162.825343 123.755201) (width 0.381) (layer F.Cu) (net 48))
+  (segment (start 162.825343 123.755201) (end 162.634923 123.945619) (width 0.381) (layer F.Cu) (net 48))
+  (segment (start 155.2956 121.886944) (end 155.2956 120.4468) (width 0.381) (layer F.Cu) (net 48))
+  (segment (start 155.2956 120.4468) (end 155.2956 120.4468) (width 0.381) (layer F.Cu) (net 48))
+  (via (at 155.2956 120.4468) (size 0.8) (drill 0.4) (layers F.Cu B.Cu) (net 48))
+  (segment (start 155.2956 103.3272) (end 159.512 99.1108) (width 0.381) (layer B.Cu) (net 48))
+  (segment (start 155.2956 120.4468) (end 155.2956 103.3272) (width 0.381) (layer B.Cu) (net 48))
   (segment (start 199.136 116.065235) (end 197.040435 118.1608) (width 0.381) (layer B.Cu) (net 49))
   (segment (start 199.136 114.808) (end 199.136 116.065235) (width 0.381) (layer B.Cu) (net 49))
@@
   (segment (start 189.1284 118.1608) (end 187.1472 120.142) (width 0.381) (layer B.Cu) (net 49))
   (segment (start 187.1472 120.142) (end 187.1472 120.142) (width 0.381) (layer B.Cu) (net 49))
-  (via (at 187.1472 120.142) (size 0.8) (drill 0.4) (layers F.Cu B.Cu) (net 49))
+  (segment (start 187.1472 120.142) (end 187.1472 122.682) (width 0.381) (layer B.Cu) (net 49))
+  (segment (start 187.1472 122.682) (end 187.1472 123.0884) (width 0.381) (layer B.Cu) (net 49))
+  (segment (start 187.1472 123.0884) (end 187.1472 123.0884) (width 0.381) (layer B.Cu) (net 49))
+  (via (at 187.1472 123.0884) (size 0.8) (drill 0.4) (layers F.Cu B.Cu) (net 49))
+  (segment (start 187.1472 123.0884) (end 162.94419 123.0884) (width 0.381) (layer F.Cu) (net 49))
+  (segment (start 157.594937 123.364609) (end 156.4132 122.182872) (width 0.381) (layer F.Cu) (net 49))
+  (segment (start 162.394262 123.36461) (end 157.594937 123.364609) (width 0.381) (layer F.Cu) (net 49))
+  (segment (start 162.94419 123.0884) (end 162.670472 123.0884) (width 0.381) (layer F.Cu) (net 49))
+  (segment (start 162.670472 123.0884) (end 162.394262 123.36461) (width 0.381) (layer F.Cu) (net 49))
+  (segment (start 156.4132 122.182872) (end 156.4132 120.4468) (width 0.381) (layer F.Cu) (net 49))
+  (segment (start 156.4132 120.4468) (end 156.4132 120.4468) (width 0.381) (layer F.Cu) (net 49))
+  (via (at 156.4132 120.4468) (size 0.8) (drill 0.4) (layers F.Cu B.Cu) (net 49))
+  (segment (start 156.4132 104.7496) (end 159.512 101.6508) (width 0.381) (layer B.Cu) (net 49))
+  (segment (start 156.4132 120.4468) (end 156.4132 104.7496) (width 0.381) (layer B.Cu) (net 49))
   (segment (start 195.961 93.205235) (end 203.5556 100.799835) (width 0.381) (layer B.Cu) (net 53))
   (segment (start 195.961 91.948) (end 195.961 93.205235) (width 0.381) (layer B.Cu) (net 53))
@@
   (segment (start 188.6712 120.0912) (end 188.6712 120.0912) (width 0.381) (layer B.Cu) (net 53))
   (via (at 188.6712 120.0912) (size 0.8) (drill 0.4) (layers F.Cu B.Cu) (net 53))
+  (segment (start 188.6712 120.0912) (end 186.2836 122.4788) (width 0.381) (layer F.Cu) (net 53))
+  (segment (start 186.2836 122.4788) (end 162.814 122.4788) (width 0.381) (layer F.Cu) (net 53))
+  (segment (start 162.814 122.4788) (end 162.4584 122.4788) (width 0.381) (layer F.Cu) (net 53))
+  (segment (start 162.4584 122.4788) (end 162.2044 122.7328) (width 0.381) (layer F.Cu) (net 53))
+  (segment (start 162.2044 122.7328) (end 162.1536 122.7836) (width 0.381) (layer F.Cu) (net 53))
+  (segment (start 162.1536 122.7836) (end 157.8356 122.7836) (width 0.381) (layer F.Cu) (net 53))
+  (segment (start 157.8356 122.7836) (end 157.4292 122.3772) (width 0.381) (layer F.Cu) (net 53))
+  (segment (start 157.4292 122.3772) (end 157.4292 120.396) (width 0.381) (layer F.Cu) (net 53))
+  (segment (start 157.4292 120.396) (end 157.4292 120.396) (width 0.381) (layer F.Cu) (net 53))
+  (via (at 157.4292 120.396) (size 0.8) (drill 0.4) (layers F.Cu B.Cu) (net 53))
+  (segment (start 157.4292 108.8136) (end 159.512 106.7308) (width 0.381) (layer B.Cu) (net 53))
+  (segment (start 157.4292 120.396) (end 157.4292 108.8136) (width 0.381) (layer B.Cu) (net 53))
   (segment (start 192.853 72.757) (end 192.8644 72.7456) (width 0.381) (layer F.Cu) (net 54))
   (segment (start 192.278 72.757) (end 192.853 72.757) (width 0.381) (layer F.Cu) (net 54))
