File: MRDT_Rover_Controller/Controller Board/Controller Board.kicad_pcb (KiCad board)
At the start: 2 copper layers, 137.6 x 81.5 mm, 31 parts, among them Q1 S8050, SW1 EG1218, U1 MCP3008

Commit message: Netlist Updated
Connections:
- 5V_Regulator1 pad 2: Net-(5V_Regulator1-Pad2) -> GND
Routing:
- net Net-(5V_Regulator1-Pad1): track 46.3 -> 28.2 mm
- net GND: track 441.8 -> 441.9 mm, vias 1 -> 2
Changed lines of the file:
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@@
     (zones 0)
     (modules 31)
-    (nets 70)
+    (nets 69)
   )
   (page A4)
@@
   (net 67 "Net-(BAT1-PadPOS)")
   (net 68 "Net-(SW1-Pad3)")
-  (net 69 "Net-(5V_Regulator1-Pad2)")
   (net_class Default "This is the default net class."
     (clearance 0.2)
@@
     (add_net "Net-(16x2_LCD1-Pad9)")
     (add_net "Net-(5V_Regulator1-Pad1)")
-    (add_net "Net-(5V_Regulator1-Pad2)")
     (add_net "Net-(BAT1-PadPOS)")
     (add_net "Net-(ESP-12E1-Pad1)")
@@
       (net 66 5V))
     (pad 2 thru_hole oval (at 2.54 0 90) (size 1.905 2) (drill 1.1) (layers *.Cu *.Mask)
-      (net 69 "Net-(5V_Regulator1-Pad2)"))
+      (net 14 GND))
     (pad 1 thru_hole rect (at 0 0 90) (size 1.905 2) (drill 1.1) (layers *.Cu *.Mask)
       (net 15 "Net-(5V_Regulator1-Pad1)"))
@@
   (segment (start 201.676 113.550765) (end 195.313235 107.188) (width 0.381) (layer B.Cu) (net 14))
   (segment (start 201.676 114.808) (end 201.676 113.550765) (width 0.381) (layer B.Cu) (net 14))
-  (segment (start 210.82 66.9036) (end 210.82 66.318) (width 0.381) (layer F.Cu) (net 14))
   (segment (start 172.5676 112.551) (end 172.5676 111.8108) (width 0.381) (layer B.Cu) (net 14))
   (segment (start 179.2224 119.2058) (end 172.5676 112.551) (width 0.381) (layer B.Cu) (net 14))
@@
   (segment (start 92.71 96.278765) (end 86.995 90.563765) (width 0.381) (layer F.Cu) (net 14))
   (segment (start 92.71 97.536) (end 92.71 96.278765) (width 0.381) (layer F.Cu) (net 14))
-  (segment (start 210.270128 65.768128) (end 210.2746 65.7726) (width 0.25) (layer F.Cu) (net 14))
-  (segment (start 210.270128 64.913472) (end 210.270128 65.768128) (width 0.25) (layer F.Cu) (net 14))
-  (segment (start 210.7692 64.4144) (end 210.270128 64.913472) (width 0.25) (layer F.Cu) (net 14))
-  (segment (start 210.82 66.318) (end 210.2746 65.7726) (width 0.381) (layer F.Cu) (net 14))
-  (segment (start 210.2746 65.7726) (end 207.494 62.992) (width 0.381) (layer F.Cu) (net 14))
+  (segment (start 210.82 64.4652) (end 210.7692 64.4144) (width 0.381) (layer F.Cu) (net 14))
+  (segment (start 210.7692 66.8922) (end 210.82 66.943) (width 0.25) (layer F.Cu) (net 14))
+  (segment (start 210.7692 64.4144) (end 210.7692 66.8922) (width 0.25) (layer F.Cu) (net 14))
+  (segment (start 210.7692 64.4144) (end 210.7692 64.4144) (width 0.381) (layer F.Cu) (net 14))
+  (via (at 210.7692 64.4144) (size 0.8) (drill 0.4) (layers F.Cu B.Cu) (net 14))
+  (segment (start 210.7692 64.4144) (end 210.1088 64.4144) (width 0.25) (layer B.Cu) (net 14))
+  (segment (start 208.6864 62.992) (end 207.01 62.992) (width 0.25) (layer B.Cu) (net 14))
+  (segment (start 210.1088 64.4144) (end 208.6864 62.992) (width 0.25) (layer B.Cu) (net 14))
   (segment (start 205.629 65.532) (end 198.517 58.42) (width 0.381) (layer F.Cu) (net 15))
   (segment (start 207.01 65.532) (end 205.629 65.532) (width 0.381) (layer F.Cu) (net 15))
@@
   (segment (start 192.8774 58.42) (end 190.9572 56.4998) (width 0.381) (layer F.Cu) (net 15))
   (segment (start 198.517 58.42) (end 192.8774 58.42) (width 0.381) (layer F.Cu) (net 15))
+  (segment (start 190.743669 54.65329) (end 190.592679 54.80428) (width 0.25) (layer F.Cu) (net 15))
+  (segment (start 191.170731 54.65329) (end 190.743669 54.65329) (width 0.25) (layer F.Cu) (net 15))
+  (segment (start 191.47271 54.955269) (end 191.170731 54.65329) (width 0.25) (layer F.Cu) (net 15))
+  (segment (start 191.47271 55.68431) (end 191.47271 54.955269) (width 0.25) (layer F.Cu) (net 15))
+  (segment (start 208.391 65.532) (end 209.6008 64.3222) (width 0.381) (layer F.Cu) (net 15))
+  (segment (start 207.01 65.532) (end 208.391 65.532) (width 0.381) (layer F.Cu) (net 15))
+  (segment (start 209.6008 63.8328) (end 210.7692 62.6644) (width 0.381) (layer F.Cu) (net 15))
+  (segment (start 209.6008 64.3222) (end 209.6008 63.8328) (width 0.381) (layer F.Cu) (net 15))
   (segment (start 167.132 109.2708) (end 163.2204 113.1824) (width 0.381) (layer F.Cu) (net 22))
   (segment (start 163.2204 113.1824) (end 163.2204 116.9416) (width 0.381) (layer F.Cu) (net 22))
@@
   (segment (start 192.532 53.3908) (end 189.6364 53.3908) (width 0.381) (layer F.Cu) (net 67))
   (segment (start 189.6364 53.3908) (end 186.683599 56.343601) (width 0.381) (layer F.Cu) (net 67))
-  (segment (start 210.7692 62.6644) (end 210.7692 60.5536) (width 0.25) (layer F.Cu) (net 15))
-  (segment (start 208.12009 57.90449) (end 200.46431 57.90449) (width 0.25) (layer F.Cu) (net 15))
-  (segment (start 210.7692 60.5536) (end 208.12009 57.90449) (width 0.25) (layer F.Cu) (net 15))
-  (segment (start 200.46431 57.90449) (end 199.60822 57.0484) (width 0.25) (layer F.Cu) (net 15))
-  (segment (start 190.743669 54.65329) (end 190.592679 54.80428) (width 0.25) (layer F.Cu) (net 15))
-  (segment (start 191.170731 54.65329) (end 190.743669 54.65329) (width 0.25) (layer F.Cu) (net 15))
-  (segment (start 191.47271 54.955269) (end 191.170731 54.65329) (width 0.25) (layer F.Cu) (net 15))
-  (segment (start 191.47271 55.68431) (end 191.47271 54.955269) (width 0.25) (layer F.Cu) (net 15))
-  (segment (start 199.60822 57.0484) (end 192.8368 57.0484) (width 0.25) (layer F.Cu) (net 15))
-  (segment (start 192.8368 57.0484) (end 191.47271 55.68431) (width 0.25) (layer F.Cu) (net 15))
 )

Commit message: Silkscreen Updated for LEDs
Parts:
- renumbered LED2 to COM, LED1 to PWR
Changed lines of the file:
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@@
   (module MRDT_Actives:LED_CREE_XLAMP_XPG (layer F.Cu)
     (at 92.71 59.69)
-    (fp_text reference LED2 (at 0.127 2.413) (layer F.SilkS)
+    (fp_text reference COM (at 0.127 2.413) (layer F.SilkS)
       (effects (font (size 0.6 0.6) (thickness 0.15)))
     )
@@
   (module MRDT_Actives:LED_CREE_XLAMP_XPG (layer F.Cu)
     (at 85.09 59.69)
-    (fp_text reference LED1 (at 0.127 2.413) (layer F.SilkS)
+    (fp_text reference PWR (at 0.127 2.413) (layer F.SilkS)
       (effects (font (size 0.6 0.6) (thickness 0.15)))
     )
