File: Rover_Controller/Rover_Controller.kicad_pcb (KiCad board)
At the start: 2 copper layers, 137.6 x 81.5 mm, 36 parts, among them Q1 S8050, SW1 SW_Push, SW2 SW_Push, SW3 SW_Push, SW4 SW_Push

Commit message: Libraries Updated & PCB Silkscreen Updated
Parts:
- renumbered 5V_Reg_1 to 5V_Reg, ADC1 to ADC, COM1 to COM, ESP-12E1 to ESP-12E, I2C_Bus1 to I2C_Bus, JP1 to JP, PWR1 to PWR, PWR_SW1 to PWR_SW, RV1 to RV, TANK1 to TANK
Other:
- board text added: "LCD Contrast"
Changed lines of the file:
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@@
   (general
     (thickness 1.6)
-    (drawings 30)
+    (drawings 31)
     (tracks 620)
     (zones 0)
@@
       (outputformat 1)
       (mirror false)
-      (drillshape 1)
+      (drillshape 0)
       (scaleselection 1)
-      (outputdirectory ""))
+      (outputdirectory "../Documentation/RemoteController_Gerbs/"))
   )
   (net 0 "")
@@
     (tags "resistor handsolder")
     (attr smd)
-    (fp_text reference R8 (at 0.113 -1.27 270) (layer F.SilkS)
+    (fp_text reference R8 (at -1.129 1.397 270) (layer F.SilkS)
       (effects (font (size 1 1) (thickness 0.15)))
     )
@@
     (tags "SOIC SO")
     (attr smd)
-    (fp_text reference I2C_Bus1 (at 0 -6.1) (layer F.SilkS)
+    (fp_text reference I2C_Bus (at 0 -6.1) (layer F.SilkS)
       (effects (font (size 1 1) (thickness 0.15)))
     )
@@
     (tags "SOIC SO")
     (attr smd)
-    (fp_text reference ADC1 (at 0 -5.9) (layer F.SilkS)
+    (fp_text reference ADC (at 0 -5.9) (layer F.SilkS)
       (effects (font (size 1 1) (thickness 0.15)))
     )
@@
     (tags "LED handsolder")
     (attr smd)
-    (fp_text reference COM1 (at 0 -1.43 90) (layer F.SilkS)
+    (fp_text reference COM (at 0 -1.43 90) (layer F.SilkS)
       (effects (font (size 1 1) (thickness 0.15)))
     )
@@
     (tags "LED handsolder")
     (attr smd)
-    (fp_text reference TANK1 (at 0 -1.43 90) (layer F.SilkS)
+    (fp_text reference TANK (at 0 -1.43 90) (layer F.SilkS)
       (effects (font (size 1 1) (thickness 0.15)))
     )
@@
     (descr "Through hole straight pin header, 1x03, 2.54mm pitch, single row")
     (tags "Through hole pin header THT 1x03 2.54mm single row")
-    (fp_text reference JP1 (at -2.54 2.286 180) (layer F.SilkS)
+    (fp_text reference JP (at -2.54 2.286 180) (layer F.SilkS)
       (effects (font (size 1 1) (thickness 0.15)))
     )
@@
   (module Rover_Controller:ESP8266_nodeMCU (layer F.Cu)
     (at 146.5072 108.4072 270)
-    (fp_text reference ESP-12E1 (at 0 -7.366 90) (layer F.SilkS)
+    (fp_text reference ESP-12E (at 0 -7.366 90) (layer F.SilkS)
       (effects (font (size 1 1) (thickness 0.15)))
     )
@@
     (tags "LED handsolder")
     (attr smd)
-    (fp_text reference PWR1 (at 0 -1.43 90) (layer F.SilkS)
+    (fp_text reference PWR (at 0 -1.43 90) (layer F.SilkS)
       (effects (font (size 1 1) (thickness 0.15)))
     )
@@
   (module 3362_Trimmer_Pot:3362P-1-103LF (layer F.Cu)
     (at 163.322 110.998)
-    (fp_text reference RV1 (at -6.8072 2.1844 90) (layer F.SilkS)
-      (effects (font (size 1 1) (thickness 0.15)))
-    )
-    (fp_text value R_POT_TRIM_10K (at -2.6924 4.826) (layer F.SilkS)
+    (fp_text reference RV (at -6.8072 2.1844 90) (layer F.SilkS)
+      (effects (font (size 1 1) (thickness 0.15)))
+    )
+    (fp_text value R_POT_TRIM_10K (at -2.286 -4.826) (layer F.SilkS)
       (effects (font (size 1 1) (thickness 0.15)))
     )
@@
     (descr "CuK miniature slide switch, OS series, SPDT, right angle, http://www.ckswitches.com/media/1428/os.pdf")
     (tags "switch SPDT")
-    (fp_text reference PWR_SW1 (at 1.524 3.302 270) (layer F.SilkS)
+    (fp_text reference PWR_SW (at 1.524 3.302 270) (layer F.SilkS)
       (effects (font (size 1 1) (thickness 0.15)))
     )
@@
     (tags "DPAK TO-252 DPAK-3 TO-252-3 SOT-428")
     (attr smd)
-    (fp_text reference 5V_Reg_1 (at 0 -4.5 90) (layer F.SilkS)
+    (fp_text reference 5V_Reg (at 0 -4.5 90) (layer F.SilkS)
       (effects (font (size 1 1) (thickness 0.15)))
     )
@@
       (rotate (xyz 0 0 0))
     )
+  )
+  (gr_text "LCD Contrast" (at 160.782 116.586) (layer F.SilkS)
+    (effects (font (size 0.762 0.762) (thickness 0.1905)))
   )
   (gr_text OFF (at 196.342 55.626 90) (layer F.SilkS)
@@
   (segment (start 194.818 63.246) (end 194.5324 62.9604) (width 0.381) (layer F.Cu) (net 58))
   (zone (net 58) (net_name +5V) (layer B.Cu) (hatch edge 0.508)
-    (connect_pads (clearance 0.508))
+    (connect_pads yes (clearance 0.508))
     (min_thickness 0.254)
     (fill yes (arc_segments 32) (thermal_gap 0.508) (thermal_bridge_width 0.508))
@@
   )
   (zone (net 13) (net_name GND) (layer F.Cu) (hatch edge 0.508)
-    (connect_pads (clearance 0.508))
+    (connect_pads yes (clearance 0.508))
     (min_thickness 0.254)
     (fill yes (arc_segments 32) (thermal_gap 0.508) (thermal_bridge_width 0.508))
     (polygon
       (pts
-        (xy 72.39 45.466) (xy 218.948 47.498) (xy 216.916 136.652) (xy 74.93 134.62) (xy 75.184 135.128)
+        (xy 218.948 47.498) (xy 216.916 136.652) (xy 75.168276 134.62341) (xy 72.39 45.466)
       )
     )
+  )
+  (zone (net 13) (net_name GND) (layer F.Cu) (hatch edge 0.508)
+    (connect_pads yes (clearance 0.508))
+    (min_thickness 0.254)
+    (fill yes (arc_segments 32) (thermal_gap 0.508) (thermal_bridge_width 0.508))
+    (polygon
+      (pts
+        (xy 75.168276 134.62341) (xy 75.184 135.128) (xy 74.93 134.62)
+      )
+    )
+  )
+  (zone (net 13) (net_name GND) (layer F.Cu) (hatch edge 0.508)
+    (connect_pads yes (clearance 0.508))
+    (min_thickness 0.254)
+    (fill yes (arc_segments 32) (thermal_gap 0.508) (thermal_bridge_width 0.508))
+    (polygon
+      (pts
+        (xy 75.168276 134.62341) (xy 75.184 135.128) (xy 74.93 134.62)
+      )
+    )
